File: interlock/relay_ctrl_lab/relay_ctrl_lab.kicad_pcb (KiCad board)
At the start: 2 copper layers, 62.2 x 33 mm, 21 parts, among them J1 RJ45_Shielded, J2 Conn_01x26, J3 Conn_01x03, J4 Conn_01x03, J5 Conn_01x02, J6 Conn_01x12, U1 TLP222A

Commit message: Fixed mistakes in interlock pcbs
Parts:
- moved J1 6.66 mm to (189.5, 135.0), turned to 180 degrees
Connections:
- J6 pad 1: Compressor2_interlock -> Backing1_active
- J6 pad 2: Backing2_interlock -> Compressor1_active
- J6 pad 3: Backing1_interlock -> Compressor2_active
- J6 pad 4: Compressor1_interlock -> Backing2_active
- J6 pad 5: Backing1_active -> Compressor2_interlock
- J6 pad 6: Compressor1_active -> Backing2_interlock
- J6 pad 7: Compressor2_active -> Backing1_interlock
- J6 pad 8: Backing2_active -> Compressor1_interlock
- R1 pad 1: Compressor2_interlock -> Backing1_active
- R2 pad 1: Backing2_interlock -> Compressor1_active
- R3 pad 1: Backing1_interlock -> Compressor2_active
- R4 pad 1: Compressor1_interlock -> Backing2_active
- R5 pad 1: Backing1_active -> Compressor2_interlock
- R6 pad 1: Compressor1_active -> Backing2_interlock
- R8 pad 1: Compressor2_active -> Backing1_interlock
- R9 pad 1: Backing2_active -> Compressor1_interlock
Routing:
- net Backing2_active: track 27.7 -> 15.5 mm
- net Compressor2_interlock: track 26.1 -> 15.7 mm
- net Compressor2_active: track 23.2 -> 15.3 mm
- net Compressor1_interlock: track 18.4 -> 24.4 mm
- net Backing1_active: track 18.6 -> 22.8 mm
- net Backing2_interlock: track 19.8 -> 15.9 mm
- net Backing1_interlock: track 18.2 -> 19.8 mm
- net Compressor1_active: track 18.8 -> 17.3 mm
- net GND: vias 0 -> 7
