File: cavity locking/NKT Basik single ended to differential modulation/NKT Basik single ended to differential modulation.kicad_pcb (KiCad board)
At the start: 2 copper layers, 29.7 x 27.2 mm, 14 parts, among them J1 Conn_01x03_Female, J2 , J3 Conn_01x02, U1 , U2 

Commit message: various
Parts:
- moved C1 10.8 mm to (157.5, 88.9), turned to 0 degrees
- moved L1 0.76 mm to (161.0, 100.4)
- moved C3 0.71 mm to (161.8, 102.6)
Routing:
- net +5V: track 11.9 -> 25.6 mm, vias 0 -> 3
Changed lines of the file:
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@@
     (thickness 1.6)
     (drawings 11)
-    (tracks 45)
+    (tracks 57)
     (zones 0)
     (modules 14)
@@
     (tags resistor)
     (attr smd)
-    (fp_text reference R1 (at 0 1.524) (layer F.SilkS)
+    (fp_text reference R1 (at -2.5145 0) (layer F.SilkS)
       (effects (font (size 1 1) (thickness 0.15)))
     )
@@
   )
   (module Inductor_SMD:L_0603_1608Metric (layer F.Cu)
-    (at 161.798 100.3555 90)
+    (at 161.036 100.3555 90)
     (descr "Inductor SMD 0603 (1608 Metric), square (rectangular) end terminal, IPC_7351 nominal, (Body size source: http://www.tortai-tech.com/upload/download/2011102023233369053.pdf), generated with kicad-footprint-generator")
     (tags inductor)
@@
   )
   (module Capacitor_SMD:C_0603_1608Metric (layer F.Cu)
-    (at 162.5345 102.616)
+    (at 161.8235 102.616)
     (descr "Capacitor SMD 0603 (1608 Metric), square (rectangular) end terminal, IPC_7351 nominal, (Body size source: http://www.tortai-tech.com/upload/download/2011102023233369053.pdf), generated with kicad-footprint-generator")
     (tags capacitor)
@@
   )
   (module Capacitor_SMD:C_0603_1608Metric (layer F.Cu)
-    (at 160.274 99.3395 90)
+    (at 157.4545 88.9)
     (descr "Capacitor SMD 0603 (1608 Metric), square (rectangular) end terminal, IPC_7351 nominal, (Body size source: http://www.tortai-tech.com/upload/download/2011102023233369053.pdf), generated with kicad-footprint-generator")
     (tags capacitor)
     (attr smd)
-    (fp_text reference C1 (at -2.286 -0.254 180) (layer F.SilkS)
-      (effects (font (size 1 1) (thickness 0.15)))
-    )
-    (fp_text value 220n (at 0 1.43 90) (layer F.Fab)
-      (effects (font (size 1 1) (thickness 0.15)))
-    )
-    (fp_text user %R (at 0 0 90) (layer F.Fab)
+    (fp_text reference C1 (at -2.286 -0.254 270) (layer F.SilkS)
+      (effects (font (size 1 1) (thickness 0.15)))
+    )
+    (fp_text value 220n (at 0 1.43) (layer F.Fab)
+      (effects (font (size 1 1) (thickness 0.15)))
+    )
+    (fp_text user %R (at 0 0) (layer F.Fab)
       (effects (font (size 0.4 0.4) (thickness 0.06)))
     )
@@
     (fp_line (start -0.8 -0.4) (end 0.8 -0.4) (layer F.Fab) (width 0.1))
     (fp_line (start -0.8 0.4) (end -0.8 -0.4) (layer F.Fab) (width 0.1))
-    (pad 2 smd roundrect (at 0.7875 0 90) (size 0.875 0.95) (layers F.Cu F.Paste F.Mask) (roundrect_rratio 0.25)
+    (pad 2 smd roundrect (at 0.7875 0) (size 0.875 0.95) (layers F.Cu F.Paste F.Mask) (roundrect_rratio 0.25)
       (net 1 +5V))
-    (pad 1 smd roundrect (at -0.7875 0 90) (size 0.875 0.95) (layers F.Cu F.Paste F.Mask) (roundrect_rratio 0.25)
+    (pad 1 smd roundrect (at -0.7875 0) (size 0.875 0.95) (layers F.Cu F.Paste F.Mask) (roundrect_rratio 0.25)
       (net 2 GND))
     (model ${KISYS3DMOD}/Capacitor_SMD.3dshapes/C_0603_1608Metric.wrl
@@
   (gr_line (start 166.878 102.362) (end 166.878 85.852) (layer Edge.Cuts) (width 0.05))
   (gr_line (start 137.16 85.852) (end 137.16 102.362) (layer Edge.Cuts) (width 0.05))
-  (segment (start 161.29 99.568) (end 160.274 98.552) (width 0.25) (layer F.Cu) (net 1))
-  (segment (start 161.798 99.568) (end 161.29 99.568) (width 0.25) (layer F.Cu) (net 1))
+  (segment (start 158.242 89.475) (end 158.242 88.9) (width 0.25) (layer F.Cu) (net 1))
+  (segment (start 158.03849 89.67851) (end 158.242 89.475) (width 0.25) (layer F.Cu) (net 1))
+  (segment (start 158.03849 91.109504) (end 158.03849 89.67851) (width 0.25) (layer F.Cu) (net 1))
+  (segment (start 157.662999 91.484995) (end 158.03849 91.109504) (width 0.25) (layer F.Cu) (net 1))
+  (segment (start 157.662999 92.5703) (end 157.662999 91.484995) (width 0.25) (layer F.Cu) (net 1))
+  (segment (start 157.93751 98.250391) (end 158.313001 97.8749) (width 0.25) (layer F.Cu) (net 1))
+  (segment (start 157.93751 99.26351) (end 157.93751 98.250391) (width 0.25) (layer F.Cu) (net 1))
+  (segment (start 158.28001 99.60601) (end 157.93751 99.26351) (width 0.25) (layer F.Cu) (net 1))
+  (segment (start 160.42299 99.60601) (end 158.28001 99.60601) (width 0.25) (layer F.Cu) (net 1))
+  (segment (start 160.461 99.568) (end 160.42299 99.60601) (width 0.25) (layer F.Cu) (net 1))
   (segment (start 158.313001 97.8749) (end 158.313001 96.9137) (width 0.25) (layer F.Cu) (net 1))
-  (segment (start 157.98749 98.200411) (end 158.313001 97.8749) (width 0.25) (layer F.Cu) (net 1))
-  (segment (start 157.98749 99.287484) (end 157.98749 98.200411) (width 0.25) (layer F.Cu) (net 1))
-  (segment (start 158.306016 99.60601) (end 157.98749 99.287484) (width 0.25) (layer F.Cu) (net 1))
-  (segment (start 159.21999 99.60601) (end 158.306016 99.60601) (width 0.25) (layer F.Cu) (net 1))
-  (segment (start 160.274 98.552) (end 159.21999 99.60601) (width 0.25) (layer F.Cu) (net 1))
-  (segment (start 157.662999 93.4324) (end 157.662999 92.5703) (width 0.25) (layer F.Cu) (net 1))
-  (segment (start 158.313001 94.082402) (end 157.662999 93.4324) (width 0.25) (layer F.Cu) (net 1))
-  (segment (start 158.313001 96.9137) (end 158.313001 94.082402) (width 0.25) (layer F.Cu) (net 1))
+  (segment (start 161.036 99.568) (end 161.036 99.568) (width 0.25) (layer F.Cu) (net 1))
+  (segment (start 161.036 99.568) (end 161.036 99.568) (width 0.25) (layer F.Cu) (net 1))
+  (via (at 161.036 99.568) (size 0.8) (drill 0.4) (layers F.Cu B.Cu) (net 1))
+  (segment (start 161.036 99.568) (end 160.461 99.568) (width 0.25) (layer F.Cu) (net 1))
+  (via (at 161.036 99.568) (size 0.8) (drill 0.4) (layers F.Cu B.Cu) (net 1))
+  (segment (start 158.242 88.9) (end 158.242 88.9) (width 0.25) (layer F.Cu) (net 1))
+  (via (at 158.242 88.9) (size 0.8) (drill 0.4) (layers F.Cu B.Cu) (net 1))
+  (segment (start 158.242 88.9) (end 160.274 88.9) (width 0.25) (layer B.Cu) (net 1))
+  (segment (start 160.274 88.9) (end 161.036 89.662) (width 0.25) (layer B.Cu) (net 1))
+  (segment (start 158.7795 88.9) (end 158.242 88.9) (width 0.7) (layer B.Cu) (net 1))
+  (segment (start 160.02 88.9) (end 158.7795 88.9) (width 0.7) (layer B.Cu) (net 1))
+  (segment (start 161.036 89.916) (end 160.02 88.9) (width 0.7) (layer B.Cu) (net 1))
+  (segment (start 161.036 99.568) (end 161.036 89.916) (width 0.7) (layer B.Cu) (net 1))
   (segment (start 152.349 96.012) (end 153.619 97.282) (width 0.25) (layer F.Cu) (net 2))
   (segment (start 151.13 96.012) (end 152.349 96.012) (width 0.25) (layer F.Cu) (net 2))
@@
   (segment (start 157.013001 90.890999) (end 157.226 90.678) (width 0.25) (layer F.Cu) (net 8))
   (segment (start 157.013001 92.5703) (end 157.013001 90.890999) (width 0.25) (layer F.Cu) (net 8))
-  (segment (start 160.909 103.454) (end 161.747 102.616) (width 0.25) (layer F.Cu) (net 9))
-  (segment (start 160.909 104.7242) (end 160.909 103.454) (width 0.25) (layer F.Cu) (net 9))
-  (segment (start 161.747 101.194) (end 161.798 101.143) (width 0.25) (layer F.Cu) (net 9))
-  (segment (start 161.747 102.616) (end 161.747 101.194) (width 0.25) (layer F.Cu) (net 9))
+  (segment (start 160.909 102.743) (end 161.036 102.616) (width 0.25) (layer F.Cu) (net 9))
+  (segment (start 160.909 104.7242) (end 160.909 102.743) (width 0.25) (layer F.Cu) (net 9))
+  (segment (start 161.036 102.616) (end 161.036 101.143) (width 0.25) (layer F.Cu) (net 9))
   (segment (start 160.833 109.7278) (end 160.909 109.6518) (width 0.25) (layer F.Cu) (net 10))
   (segment (start 160.833 112.014) (end 160.833 109.7278) (width 0.25) (layer F.Cu) (net 10))
