File: cavity locking/stemlab cavity locking/red_pitaya_shield/output_amplifier.sch (KiCad schematic (older format))
At the start: 20 parts, among them J1 Conn_Coaxial, J2 Conn_Coaxial, J9 Conn_01x02, U1 LM4120AIM5-5.0_NOPB, U2 LP2985-10.0, U3 ADA4841-1YRJZ-R7

Commit message: Pitaya updates
Parts:
- C2: value C -> 10n
Changed lines of the file:
@@
 AR Path="/5EF07A16/5EF22F61" Ref="C2"  Part="1"
 F 0 "C2" H 5265 2496 50  0000 L CNN
-F 1 "C" H 5265 2405 50  0000 L CNN
+F 1 "10n" H 5265 2405 50  0000 L CNN
 F 2 "Capacitor_SMD:C_0805_2012Metric" H 5188 2300 50  0001 C CNN
 F 3 "~" H 5150 2450 50  0001 C CNN
