File: tec control/mtd415te/rev 3.0/mtd415te.sch (KiCad schematic (older format))
At the start: 30 parts, among them J1 Conn_02x04_Odd_Even, J10 DB9_Female_MountingHoles, J11 DB9_Female_MountingHoles, J12 Conn_02x04_Odd_Even, J13 Conn_02x04_Odd_Even, J14 Conn_02x04_Odd_Even, J2 EJ503A, J3 Conn_01x08, J4 Conn_01x08, J5 Conn_01x04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

Commit message: Add tec control pcbs
Parts:
- removed C1, C2: 0.1uF, Capacitor_SMD:C_0603_1608Metric, symbol Device:C
- removed J12, J9: Conn_02x04_Odd_Even, Connector_PinHeader_2.54mm:PinHeader_2x04_P2.54mm_Vertical, symbol Connector_Generic:Conn_02x04_Odd_Even
- removed R3, R4: PULLDOWN, Resistor_SMD:R_0805_2012Metric, symbol Device:R
- removed U2: TXS0108EPWR, footprints:TXS0108EPWR, symbol TXS0108EPWR:TXS0108EPWR
- added C1, C2: CP1_Small, Capacitor_SMD:C_0805_2012Metric, symbol Device:CP1_Small
- added J12, J15: Conn_01x06, Connector_PinHeader_2.54mm:PinHeader_1x06_P2.54mm_Vertical, symbol Connector_Generic:Conn_01x06
- added J9: Conn_01x04, Connector_PinHeader_2.54mm:PinHeader_1x04_P2.54mm_Vertical, symbol Connector_Generic:Conn_01x04
Connections:
- net labels added: BUTTON4, STATUS1, STATUS2, TEC1_S+, TEC1_S-, TEC2_S+, TEC2_S-
- net labels removed: 3V3_GND1, 3V3_GND2, 3V3_GND3, 3V3_GND4, CYCLINGBUTTON, ENABLE1_C, ENABLE2_C, RX1_C, RX2_C, STATUS1_C, STATUS2_C, TX1_C, TX2_C
- wire segments 26 -> 20
Other:
- moved on the sheet: J11, J5
