File: tec control/mtd415te/rev 4.0/mtd415te.sch (KiCad schematic (older format))
At the start: 26 parts, among them J1 Conn_02x04_Odd_Even, J10 DB9_Female_MountingHoles, J11 DB9_Female_MountingHoles, J13 Conn_02x04_Odd_Even, J14 Conn_02x04_Odd_Even, J2 EJ503A, J3 Conn_01x08, J4 Conn_01x08, J5 Conn_01x04, J6 Conn_01x08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

Commit message: Add tec control pcbs
Parts:
- removed C? (x2): CP1_Small, Capacitor_SMD:C_0805_2012Metric, symbol Device:CP1_Small
- removed J9: Conn_01x04, Connector_PinHeader_2.54mm:PinHeader_1x04_P2.54mm_Vertical, symbol Connector_Generic:Conn_01x04
- removed U1: Teensy4.0, footprints:Teensy40, symbol teensy:Teensy4.0
- added J12, J9: Conn_02x04_Odd_Even, Connector_PinHeader_2.54mm:PinHeader_2x04_P2.54mm_Vertical, symbol Connector_Generic:Conn_02x04_Odd_Even
- added R3, R4: PULLDOWN, Resistor_SMD:R_0805_2012Metric, symbol Device:R
- added U1: Teensy3.6, footprints:Teensy35_36, symbol teensy:Teensy3.6
Connections:
- net labels added: 3V3_GND1, 3V3_GND2, 3V3_GND3, 3V3_GND4, CYCLINGBUTTON
- net labels removed: BUTTON4
Other:
- moved on the sheet: J5
