File: PXIe5171 PFI breakout/PXIe5171 PFI breakout.sch (KiCad schematic (older format))
At the start: 14 parts, among them J1 Conn_Coaxial, J10 2013978-1, J2 Conn_Coaxial, J3 Conn_Coaxial, J4 Conn_Coaxial, J5 Conn_Coaxial, J6 Conn_Coaxial, J7 Conn_Coaxial, J8 Conn_Coaxial, J9 Conn_Coaxial

Commit message: Removed superfluous libraries
Parts:
- H1, H2, H3, H4: symbol Mechanical:MountingHole_Pad -> PXIe5171-PFI-breakout-rescue:MountingHole_Pad-Mechanical
- J1, J2, J3, J4, J5, J6, J7, J8, J9: symbol Connector:Conn_Coaxial -> PXIe5171-PFI-breakout-rescue:Conn_Coaxial-Connector
Changed lines of the file:
@@
 $EndDescr
 $Comp
-L Mechanical:MountingHole_Pad H2
+L PXIe5171-PFI-breakout-rescue:MountingHole_Pad-Mechanical H2
 U 1 1 5E8517BC
 P 9400 3750
@@
 $EndComp
 $Comp
-L Mechanical:MountingHole_Pad H1
+L PXIe5171-PFI-breakout-rescue:MountingHole_Pad-Mechanical H1
 U 1 1 5E853D93
 P 9400 5850
@@
 $EndComp
 $Comp
-L Mechanical:MountingHole_Pad H3
+L PXIe5171-PFI-breakout-rescue:MountingHole_Pad-Mechanical H3
 U 1 1 5E85724D
 P 10700 4100
@@
 $EndComp
 $Comp
-L Mechanical:MountingHole_Pad H4
+L PXIe5171-PFI-breakout-rescue:MountingHole_Pad-Mechanical H4
 U 1 1 5EED193D
 P 10100 2800
@@
 $EndComp
 $Comp
-L Connector:Conn_Coaxial J1
+L PXIe5171-PFI-breakout-rescue:Conn_Coaxial-Connector J1
 U 1 1 5F705123
 P 1250 900
@@
 $EndComp
 $Comp
-L power:GND #PWR0101
+L PXIe5171-PFI-breakout-rescue:GND-power #PWR0101
 U 1 1 5F705D84
 P 1250 1100
@@
 PFI0
 $Comp
-L Connector:Conn_Coaxial J2
+L PXIe5171-PFI-breakout-rescue:Conn_Coaxial-Connector J2
 U 1 1 5F7063EC
 P 1250 1450
@@
 $EndComp
 $Comp
-L power:GND #PWR0102
+L PXIe5171-PFI-breakout-rescue:GND-power #PWR0102
 U 1 1 5F7063F2
 P 1250 1650
@@
 PFI1
 $Comp
-L Connector:Conn_Coaxial J3
+L PXIe5171-PFI-breakout-rescue:Conn_Coaxial-Connector J3
 U 1 1 5F7078CD
 P 1250 2000
@@
 $EndComp
 $Comp
-L power:GND #PWR0103
+L PXIe5171-PFI-breakout-rescue:GND-power #PWR0103
 U 1 1 5F7078D3
 P 1250 2200
@@
 PFI2
 $Comp
-L Connector:Conn_Coaxial J4
+L PXIe5171-PFI-breakout-rescue:Conn_Coaxial-Connector J4
 U 1 1 5F7078DA
 P 1250 2550
@@
 $EndComp
 $Comp
-L power:GND #PWR0104
+L PXIe5171-PFI-breakout-rescue:GND-power #PWR0104
 U 1 1 5F7078E0
 P 1250 2750
@@
 PFI3
 $Comp
-L Connector:Conn_Coaxial J5
+L PXIe5171-PFI-breakout-rescue:Conn_Coaxial-Connector J5
 U 1 1 5F70CF85
 P 1250 3100
@@
 $EndComp
 $Comp
-L power:GND #PWR0105
+L PXIe5171-PFI-breakout-rescue:GND-power #PWR0105
 U 1 1 5F70CF8B
 P 1250 3300
@@
 PFI4
 $Comp
-L Connector:Conn_Coaxial J6
+L PXIe5171-PFI-breakout-rescue:Conn_Coaxial-Connector J6
 U 1 1 5F70CF92
 P 1250 3650
@@
 $EndComp
 $Comp
-L power:GND #PWR0106
+L PXIe5171-PFI-breakout-rescue:GND-power #PWR0106
 U 1 1 5F70CF98
 P 1250 3850
@@
 PFI5
 $Comp
-L Connector:Conn_Coaxial J7
+L PXIe5171-PFI-breakout-rescue:Conn_Coaxial-Connector J7
 U 1 1 5F70CF9F
 P 1250 4200
@@
 $EndComp
 $Comp
-L power:GND #PWR0107
+L PXIe5171-PFI-breakout-rescue:GND-power #PWR0107
 U 1 1 5F70CFA5
 P 1250 4400
@@
 PFI6
 $Comp
-L Connector:Conn_Coaxial J8
+L PXIe5171-PFI-breakout-rescue:Conn_Coaxial-Connector J8
 U 1 1 5F70CFAC
 P 1250 4750
@@
 $EndComp
 $Comp
-L power:GND #PWR0108
+L PXIe5171-PFI-breakout-rescue:GND-power #PWR0108
 U 1 1 5F70CFB2
 P 1250 4950
@@
 CLC_IN
 $Comp
-L Connector:Conn_Coaxial J9
+L PXIe5171-PFI-breakout-rescue:Conn_Coaxial-Connector J9
 U 1 1 5F70DD54
 P 1250 5400
@@
 $EndComp
 $Comp
-L power:GND #PWR0109
+L PXIe5171-PFI-breakout-rescue:GND-power #PWR0109
 U 1 1 5F70DD5A
 P 1250 5600
@@
 $EndComp
 $Comp
-L power:GND #PWR0110
+L PXIe5171-PFI-breakout-rescue:GND-power #PWR0110
 U 1 1 5F7106EE
 P 4200 1250
@@
 $EndComp
 $Comp
-L power:GND #PWR0111
+L PXIe5171-PFI-breakout-rescue:GND-power #PWR0111
 U 1 1 5F71115E
 P 4200 1450
@@
 Connection ~ 4200 1450
 $Comp
-L power:GND #PWR0112
+L PXIe5171-PFI-breakout-rescue:GND-power #PWR0112
 U 1 1 5F7117A3
 P 4200 1750
@@
 Connection ~ 4200 1750
 $Comp
-L power:GND #PWR0113
+L PXIe5171-PFI-breakout-rescue:GND-power #PWR0113
 U 1 1 5F71210F
 P 4200 2150
@@
 $EndComp
 $Comp
-L power:GND #PWR0114
+L PXIe5171-PFI-breakout-rescue:GND-power #PWR0114
 U 1 1 5F712588
 P 4200 2450
@@
 $EndComp
 $Comp
-L power:GND #PWR0115
+L PXIe5171-PFI-breakout-rescue:GND-power #PWR0115
 U 1 1 5F712D19
 P 4200 3050
@@
 $EndComp
 $Comp
-L power:GND #PWR0116
+L PXIe5171-PFI-breakout-rescue:GND-power #PWR0116
 U 1 1 5F713301
 P 4200 3250
@@
 CLC_OUT
 $Comp
-L power:GND #PWR?
+L PXIe5171-PFI-breakout-rescue:GND-power #PWR?
 U 1 1 5F73130F
 P 9500 5850
@@
 $EndComp
 $Comp
-L power:GND #PWR?
+L PXIe5171-PFI-breakout-rescue:GND-power #PWR?
 U 1 1 5F731F11
 P 9500 3750
@@
 $EndComp
 $Comp
-L power:GND #PWR?
+L PXIe5171-PFI-breakout-rescue:GND-power #PWR?
 U 1 1 5F732067
 P 10200 2800
@@
 $EndComp
 $Comp
-L power:GND #PWR?
+L PXIe5171-PFI-breakout-rescue:GND-power #PWR?
 U 1 1 5F732500
 P 10800 4100
